Commit message: repair collision boundaries

File: src/bot_description/urdf/bot.urdf (robot description, URDF)
Before this commit: robot bot, 5 links, 4 joints
Links:
- link caster_40mm_wheel_support_01: geometry collision box size=0.04 0.04 0.02; visual mesh filename=package://bot_description/meshes/caster_40mm_wheel_support_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
- link wheel: geometry collision cylinder length=0.04 radius=0.033; visual mesh filename=package://bot_description/meshes/tt_motor_3777_v10__8.stl
- link wheel_2: geometry collision cylinder length=0.04 radius=0.033; visual mesh filename=package://bot_description/meshes/tt_motor_3777_v10__8.stl

Commit message: reduced spacers and added dummy_link

File: src/bot_description/urdf/bot.urdf (robot description, URDF)
Before this commit: robot bot, 5 links, 4 joints
Links:
- added link base_link
- link caster_40mm_wheel_30mm_01: geometry collision sphere radius=0.015; visual mesh filename=package://bot_description/meshes/caster_40mm_wheel_30mm_01.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
- link chassis: mass 0.339643 -> 0.339156
Joints:
- added joint base_joint: type fixed, parent base_link, child chassis
- joint caster_swivel: origin xyz=0.0967499 -2.63931e-05 -0.0186507 rpy=0 -0 -1.5708 -> xyz=0.0967499 -2.63931e-05 -0.0116507 rpy=0 -0 -1.5708
- joint right_wheel: origin xyz=-0.00036815 -0.0387764 -0.0135492 rpy=-1.5708 -0 0 -> xyz=-0.00036815 -0.0387764 -0.0135492 rpy=1.5708 -0.995712 -3.14159
