Commit message: Added mpu6050 to CAD and URDF

File: src/bot_description/urdf/bot.urdf (robot description, URDF)
Before this commit: robot bot, 6 links, 5 joints
Links:
- added link imu_link, mass 1e-9
- link chassis: mass 0.339156 -> 0.339243; geometry collision box size=0.19 0.10 0.04; visual mesh filename=package://bot_description/meshes/bateria_18650.stl
Joints:
- added joint imu_link_frame: type fixed, parent chassis, child imu_link, origin xyz=0.0979786 0.033993 0.0089771 rpy=0 -0 0, axis 0 0 0
- joint caster_swivel: origin xyz=0.0967499 -2.63931e-05 -0.0116507 rpy=0 -0 -1.5708 -> xyz=0.0967499 -2.63931e-05 -0.0129007 rpy=-0 0 1.71597
- joint caster_wheel: origin xyz=-0 -0.0155 -0.02 rpy=1.5708 0 1.5708 -> xyz=-0 -0.0155 -0.02 rpy=1.5708 -0 1.5708
